Commit message: add plugin

File: src/Robot_Mecanum_description/urdf/Robot_Mecanum.urdf.xacro (robot description, xacro)
@@ -7,3 +7,4 @@
     <xacro:include filename="camera.xacro"/>
     <xacro:include filename="lidar.xacro"/>
+    <xacro:include filename="imu.xacro"/>
 </robot>

File: src/Robot_Mecanum_description/urdf/Robot_Mecanum.xacro (robot description, xacro)
@@ -258,24 +258,4 @@
     <geometry>
       <mesh filename="file://$(find Robot_Mecanum_description)/meshes/Pokrywa_1.stl" scale="0.001 0.001 0.001"/>
-    </geometry>
-  </collision>
-</link>
-<link name="JetsonNano_1">
-  <inertial>
-    <origin xyz="0.04569099999999997 1.744770795704311e-07 -0.007500491924311237" rpy="0 0 0"/>
-    <mass value="1.884"/>
-    <inertia ixx="0.001146" iyy="0.001711" izz="0.002575" ixy="0.0" iyz="0.0" ixz="0.0"/>
-  </inertial>
-  <visual>
-    <origin xyz="0.066382 -0.000802 -0.081321" rpy="0 0 0"/>
-    <geometry>
-      <mesh filename="file://$(find Robot_Mecanum_description)/meshes/JetsonNano_1.stl" scale="0.001 0.001 0.001"/>
-    </geometry>
-    <material name="gray"/>
-  </visual>
-  <collision>
-    <origin xyz="0.066382 -0.000802 -0.081321" rpy="0 0 0"/>
-    <geometry>
-      <mesh filename="file://$(find Robot_Mecanum_description)/meshes/JetsonNano_1.stl" scale="0.001 0.001 0.001"/>
     </geometry>
   </collision>
@@ -445,9 +425,4 @@
   <parent link="Stelarz_1"/>
   <child link="Pokrywa_1"/>
-</joint>
-<joint name="Sztywne 33" type="fixed">
-  <origin xyz="0.019309 0.040802 0.0255" rpy="0 0 0"/>
-  <parent link="Pokrywa_1"/>
-  <child link="JetsonNano_1"/>
 </joint>
 <joint name="Obrot 35" type="continuous">

File: src/Robot_Mecanum_description/urdf/camera.xacro (robot description, xacro)
@@ -26,3 +26,20 @@
         <child link="Kamera_1"/>
     </joint>
+    <link name = "Camera"></link>
+    <joint name="Camera_joint" type="fixed">
+        <origin xyz="0.06 0 -0.03" rpy="0 -0.34 0"/>
+        <parent link="Kamera_1"/>
+        <child link="Camera"/>
+    </joint>
+    <gazebo reference = "Camera">
+        <material>Gazebo/Red</material>
+        <sensor name="camera_sensor" type="camera">
+            <pose>0 0 0 0 0 0</pose>
+            <visualize>true</visualize>
+            <update_rate>10.0</update_rate>
+            <plugin name="camera_controller" filename="libgazebo_ros_camera.so">
+                <frame_name>camera_link</frame_name>
+            </plugin>
+        </sensor>
+    </gazebo>
 </robot>

File: src/Robot_Mecanum_description/urdf/lidar.xacro (robot description, xacro)
@@ -25,4 +25,38 @@
         <parent link="Dach_1"/>
         <child link="Lidar_1"/>
-      </joint>
+    </joint>
+    <gazebo reference="Lidar_1">
+      <sensor name="laser" type="ray">
+          <pose> 0 0 0 0 0 0 </pose>
+          <visualize>true</visualize>
+          <update_rate>10</update_rate>
+          <ray>
+              <scan>
+                  <horizontal>
+                      <samples>360</samples>
+                      <resolution>1</resolution>
+                      <min_angle>-3.14</min_angle>
+                      <max_angle>3.14</max_angle>
+                  </horizontal>
+              </scan>
+              <range>
+                  <min>0.3</min>
+                  <max>12</max>
+                  <resolution>0.01</resolution>
+              </range>
+              <noise>
+                  <type>gaussian</type>
+                  <mean>0.0</mean>
+                  <stddev>0.01</stddev>
+                </noise>
+          </ray>
+          <plugin name="lidar" filename="libgazebo_ros_ray_sensor.so">
+              <ros>
+                  <remapping>~/out:=scan</remapping>
+              </ros>
+              <output_type>sensor_msgs/LaserScan</output_type>
+              <frame_name>lidar_link</frame_name>
+          </plugin>
+      </sensor>
+    </gazebo>
 </robot>
