Commit message: add control

File: src/Robot_Mecanum_description/urdf/Robot_Mecanum.xacro (robot description, xacro)
@@ -430,5 +430,5 @@
   <parent link="Silnik2_1"/>
   <child link="Kolo2_1"/>
-  <axis xyz="0.0 -1.0 0.0"/>
+  <axis xyz="0.0 1.0 0.0"/>
 </joint>
 <joint name="Obrot 36" type="continuous">
@@ -442,5 +442,5 @@
   <parent link="Silnik4_1"/>
   <child link="Kolo4_1"/>
-  <axis xyz="0.0 -1.0 0.0"/>
+  <axis xyz="0.0 1.0 0.0"/>
 </joint>
 <joint name="Obrot 38" type="continuous">
